File: voltai_card.kicad_pcb (KiCad board)
At the start: 2 copper layers, 89 x 51 mm, 3 parts, among them U1 ST25DV64KC-JF6D3

Commit message: my branch
Connections:
- U1 pad 3: unconnected-(U1-V_EH-Pad3) -> Net-(U1-V_EH)
- U1 pad 6: unconnected-(U1-VSS-Pad6) -> Net-(U1-VSS)
Other:
- board text added: "Johan Vlassak"
- board text added: "Software Engineer"
- board text removed: "Applications Engineer"
- board text removed: "Fengrui Zuo"
- board text removed: "designed by voltai.ai"
